File: NGCL.kicad_sch (KiCad schematic)
At the start: 6 parts, among them U1 BQ24166

Commit message: add some passives and audio connector
Parts:
- removed R1, R2, R3, R4, R5: 10k, NGCL_Passive:RES0603, symbol NGCL_Passive:RES0603-10k-1
- removed U1: BQ24166, NGCL_IC-Power:QFN50P410X410X100-24P, symbol NGCL_IC-Power:BQ24166RGER
Connections:
- no-connect marks 15 -> 0
